File: V1_21_03_2023/V1_21_03_2023.kicad_sch (KiCad schematic)
At the start: 12 parts, among them J1 USB_B_Micro, Q1 UMH3N, U1 ESP32-PICO-D4, U2 CP2104, Y1 RV-8803-C7-TA-QC

Commit message: Pruebas conexion de cables
Parts:
- added AE1: Antenna_Shield, RF_Antenna:Texas_SWRA117D_2.4GHz_Right, symbol Device:Antenna_Shield
- added C10, C11, C4, C5, C6, C7, C9: 1uF/50V, Capacitor_SMD:C_0201_0603Metric, symbol Device:C
- added C12, C14: 4.7uF/25V, Capacitor_SMD:C_0201_0603Metric, symbol Device:C
- added C13: 1Uf/50V, Capacitor_SMD:C_0201_0603Metric, symbol Device:C
- added C8: C, Capacitor_SMD:C_0201_0603Metric, symbol Device:C
- added D2, D3, D4: MBR0530, Diode_SMD:D_SOD-123, symbol Diode:MBR0530
- added J2: Conn_01x24, Connector_Molex:Molex_SL_171971-0024_1x24_P2.54mm_Vertical, symbol Connector_Generic:Conn_01x24
- added L1: L, Inductor_SMD:L_6.3x6.3_H3, symbol Device:L
- added Q2: Si2371EDS, Package_TO_SOT_SMD:SOT-23, symbol Transistor_FET:Si2371EDS
- added R10, R11: 100K, Resistor_SMD:R_0402_1005Metric, symbol Device:R
- added R4, R5, R6, R7, R8: 10K, Resistor_SMD:R_0201_0603Metric, symbol Device:R
- added R9: 0.14R, Resistor_SMD:R_0201_0603Metric, symbol Device:R
- added SW1, SW2, SW3, SW4: SW_Push, Button_Switch_SMD:SW_SPST_CK_RS282G05A3, symbol Switch:SW_Push
- C1: value C -> 0.1uF; footprint (none) -> Capacitor_SMD:C_0201_0603Metric
- C2: value C -> 1uF; footprint (none) -> Capacitor_SMD:C_0201_0603Metric
- C3: value C -> 10uF; footprint (none) -> Capacitor_SMD:C_0201_0603Metric
- J1: footprint (none) -> Connector_USB:USB_Micro-AB_Molex_47590-0001
- R1, R2, R3: value R -> 10K; footprint (none) -> Resistor_SMD:R_0201_0603Metric
- Y1: footprint MICROCRYSTAL_RV-8803-C7-TA-QC -> RV-8803:MICROCRYSTAL_RV-8803-C7-TA-QC
Connections:
- net +3.3V: now also C14.1, C6.2, J2.10 (Pin_10), J2.9 (Pin_9), L1.2, R10.1, SW1.2, SW2.2, SW3.2, SW4.2; no longer C2.2, D1.4 (K), J1.1 (VBUS), U2.7 (REGIN), U2.8 (VBUS)
- net 0: now also C10.1, C11.1, C13.2, C14.2, C4.1, C5.1, C6.1, C7.1, C8.1, C9.1, D3.1 (K), J2.17 (Pin_17), J2.8 (Pin_8), R11.2, R8.2, R9.2
- net SW_3: now reaches U1.10 (IO34)
- net SW_3: now also R6.2, SW3.1
- net SW_1: now reaches U1.11 (IO35)
- net SW_1: now also R4.2, SW1.1
- net ADC_BATT: now reaches U1.13 (IO33)
- net ADC_BATT: now also R10.2, R11.1
- net SW_2: now reaches U1.14 (IO25)
- net SW_2: now also R5.2, SW2.1
- net ACC_INT1: now reaches U1.17 (IO14)
- net ACC_INT2: now reaches U1.18 (IO12)
- net at U1.2 (LNA_IN): now also AE1.1 (A)
- net SW_4: now reaches U1.24 (IO4)
- net SW_4: now also R7.2, SW4.1
- net RES: now reaches U1.28 (SD2/IO9)
- net RES: now also J2.15 (Pin_15)
- net DC: now reaches U1.29 (SD3/IO10)
- net DC: now also J2.14 (Pin_14)
- net SS: now reaches U1.34 (IO5)
- net SS: now also J2.13 (Pin_13)
- net SCK: now reaches U1.35 (IO18)
- net SCK: now also J2.12 (Pin_12)
- net MOSI: now reaches U1.36 (IO23)
- net MOSI: now also J2.11 (Pin_11)
- net BUSY: now reaches U1.38 (IO19)
- net BUSY: now also J2.16 (Pin_16)
- new net: C11.2, J2.3 (Pin_3)
- new net: C10.2, J2.1 (Pin_1)
- new net: C5.2, J2.20 (Pin_20)
- new net: C4.2, J2.21 (Pin_21)
- new net: C9.2, J2.5 (Pin_5)
- new net: C8.2, J2.6 (Pin_6)
- new net: C7.2, J2.7 (Pin_7)
- new net: C12.2, D4.2 (A), L1.1, Q2.3 (D)
- new net: C12.1, D2.1 (K), D3.2 (A)
- new net GDR: J2.23 (Pin_23), Q2.1 (G), R8.1
- new net GND: AE1.2 (Shield), R4.1, R5.1, R6.1, R7.1
- new net PREVGH: C13.1, D4.1 (K), J2.4 (Pin_4)
- new net PREVGL: D2.2 (A), J2.2 (Pin_2)
- new net RESET: J2.22 (Pin_22), Q2.2 (S), R9.1
- new net VBUS: C2.2, D1.4 (K), J1.1 (VBUS), U2.7 (REGIN), U2.8 (VBUS)
- no-connect marks 26 -> 32
Other:
- note added: "Conector"
